Commit message: add customized-urdf with new bumpers

File: husky_custom_description/urdf/custom_description.urdf.xacro (robot description, xacro)
@@ -21,11 +21,17 @@
 ARISING IN ANY WAY OUT OF THE USE OF THIS SOFTWARE, EVEN IF ADVISED OF THE POSSIBILITY OF SUCH DAMAGE.
 -->
-<robot name="husky" xmlns:xacro="http://ros.org/wiki/xacro">
-  <xacro:arg name="laser_enabled" default="$(optenv HUSKY_LMS1XX_ENABLED false)" />
+<!-- <robot name="husky" xmlns:xacro="http://ros.org/wiki/xacro"> -->
+<robot xmlns:xacro="http://ros.org/wiki/xacro">
+  <!-- <xacro:arg name="laser_enabled" default="$(optenv HUSKY_LMS1XX_ENABLED false)" />
   <xacro:arg name="ur5_enabled" default="$(optenv HUSKY_UR5_ENABLED false)" />
-  <xacro:arg name="kinect_enabled" default="false" />
-  <xacro:include filename="$(find husky_description)/urdf/husky.urdf.xacro" />
-  <xacro:husky_robot />
+  <xacro:arg name="kinect_enabled" default="false" /> -->
+  <!-- <xacro:include filename="$(find husky_description)/urdf/husky.urdf.xacro" /> -->
+  <!-- <xacro:husky_robot /> -->
   <!-- Insert customization below, sample provided: -->
+  <!-- circular bumper Properties -->
+  <xacro:property name="circular_bumper_length" value="0.1" />
+  <xacro:property name="circular_bumper_radius" value="0.15" />
+  <xacro:property name="circular_bumper_enable"    value="$(optenv CIRCULAR_BUMPER 1)" />
+  <xacro:property name="planar_bumper_enable"     value="$(optenv PLANAR_BUMPER 0)" />
   <link name="bowler_link">
     <visual>
@@ -46,3 +52,45 @@
     <origin xyz="0.1 -0.1 0" rpy="0 0 0.5" />
   </joint>
+  <xacro:if value="${circular_bumper_enable}">
+    <link name="circular_bumper_link">
+      <visual>
+      <material name="black"/>
+        <geometry>
+          <mesh filename="package://husky_custom_description/meshes/circle_bumper.STL" />
+        </geometry>
+      </visual>
+      <collision>
+        <origin xyz="0.15 0.05 0.15" rpy="1.5707 0 0" />
+        <geometry>
+          <cylinder length="${circular_bumper_length}" radius="${circular_bumper_radius}" />
+        </geometry>
+      </collision>
+    </link>
+    <joint name="circular_bumper_joint" type="fixed">
+      <parent link="base_link" />
+      <child link="circular_bumper_link" />
+      <origin xyz="0.22 -0.15 0.0" rpy="-1.5707 0 0" />
+    </joint>
+    </xacro:if>
+  <xacro:if value="${planar_bumper_enable}">
+    <link name="planar_bumper_link">
+      <visual>
+      <material name="black"/>
+        <geometry>
+          <mesh filename="package://husky_custom_description/meshes/planar_bumper.STL" />
+        </geometry>
+      </visual>
+      <collision>
+        <origin xyz="0.15 0.15 0.05" rpy="0 0 0" />
+        <geometry>
+          <box size="0.3 0.3 0.1" rpy="0 0 0"/>
+        </geometry>
+      </collision>
+    </link>
+    <joint name="planar_bumper_joint" type="fixed">
+      <parent link="base_link" />
+      <child link="planar_bumper_link" />
+      <origin xyz="0.5 -0.15 -0.1" rpy="0 0 1.5707" />
+    </joint>
+    </xacro:if>
 </robot>
